File: Pregnant Laser Mouse.kicad_sch (KiCad schematic)
At the start: 27 parts, among them J1 Amiga_Conn, J2 Conn_01x01, M1 ADNS-9800, Q1 IRLML6302TRPBF, SW1 LEFT, SW2 MID, SW3 RIGHT, SW4 RESET, U1 SeeeduinoXIAO, U2 LT1963AxST-3.3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

Commit message: Tidy Up
Code update
Silk update
General Tidy
Parts:
- added JP1, JP2, JP3: ~, Jumper:SolderJumper-3_P1.3mm_Bridged12_Pad1.0x1.5mm, symbol Jumper:SolderJumper_3_Bridged12
- C1, C5, C6, C7: Digikey (none) -> 399-C0805C104K5RAC7210CT-ND
- C2: Digikey (none) -> 399-C0805C471K5RAC7800CT-ND
- C3, C9: Digikey (none) -> 399-C0805C106K8PAC7800CT-ND
- C4: Digikey (none) -> 399-C0805C105K4RAC7800CT-ND
- C8: Digikey (none) -> 399-C0805C335K8PAC7800CT-ND
- J1: Digikey (none) -> 2057-PH1-10-UA-ND
- J2: value Conn_01x01 -> Reset Hole; now not fitted; now left out of the parts list
- M1: Digikey (none) -> Aliexpress Get Lens Also
- Q1: Digikey (none) -> IRLML6302PBFCT-ND / DMG2301LK-7DICT-ND
- R1, R2, R3: Digikey (none) -> 2019-RK73H2ATTD1801FCT-ND
- R4, R5, R6: Digikey (none) -> 2019-RK73H2ATTD3301FCT-ND
- SW1, SW2, SW3: Availability In Stock -> (none); Check_prices https://www.snapeda.com/parts/D2F-01F/Omron+Electronics+Inc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 -> (none); Description_1 Ultra Subminiature Basic Switch,Snap Action, Pin Plunger, .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 -> (none); Digikey (none) -> SW501-ND; MANUFACTURER Omron -> (none); MAXIMUM_PACKAGE_HEIGHT 7.8 mm -> (none); MF Omron Electronics -> (none); MP D2F-01F -> (none); PARTREV B036-E1-12 -> (none); Package None -> (none); Price None -> (none); SNAPEDA_PN D2F-01F -> (none); STANDARD Manufacturer Recommendations -> (none); SnapEDA_Link https://www.snapeda.com/parts/D2F-01F/Omron+Electronics+Inc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 -> (none)
- SW4: Digikey (none) -> 450-1650-ND
- U1: Digikey (none) -> 1597-102010328-ND
- U2: Digikey (none) -> AP7361C-33E-13DICT-ND
- U3, U4: Digikey (none) -> 1727-4578-1-ND
Connections:
- net GND: now also JP1.2 (C), JP2.2 (C), JP3.2 (C); no longer SW1.1, SW2.1, SW3.1
- net SW2_GND3: now reaches SW2.3
- net SW2_GND3: now also JP2.3 (B)
- net SW1_GND3: now reaches SW1.3
- net SW1_GND3: now also JP1.3 (B)
- net SW3_GND3: now reaches SW3.3
- net SW3_GND3: now also JP3.3 (B)
- new net SW1_GND1: JP1.1 (A), SW1.1
- new net SW2_GND1: JP2.1 (A), SW2.1
- new net SW3_GND1: JP3.1 (A), SW3.1
- no-connect marks 11 -> 8
Other:
- company: (none) -> Board Folk 2024
- title: (none) -> Amiga Pregnant Laser Mouse

Commit message: Update to 1.1
Removed solder bridges to allow switch to be used on either side without having to cut and rebridge
Parts:
- removed JP1, JP2, JP3: ~, Jumper:SolderJumper-3_P1.3mm_Bridged12_Pad1.0x1.5mm, symbol Jumper:SolderJumper_3_Bridged12
Connections:
- net SW1_GND1 is gone; now on net GND: SW1.1
- net SW1_GND3 is gone; now on net GND: SW1.3
- net SW2_GND1 is gone; now on net GND: SW2.1
- net SW2_GND3 is gone; now on net GND: SW2.3
- net SW3_GND1 is gone; now on net GND: SW3.1
- net SW3_GND3 is gone; now on net GND: SW3.3
